Commit message: updated arm URDF to have a 'base', 'circle' and first arm linkage, should complete arm, and find way to have less 'magic numbers'

File: description/arm.urdf.xacro (robot description, xacro)
@@ -4,8 +4,14 @@
         <color rgba="1 1 1 1"/>
     </material>
+    <material name="blue">
+        <color rgba="0 0 1 1"/>
+    </material>
+    <material name="red">
+        <color rgba="1 0 0 1"/>
+    </material>
     <!-- Base link, true, non-relative 0,0,0 of world -->
     <link name="world"></link>
     <!-- connection from the world, to the base of the arm-->
-    <joint name="base_joint" type="fixed">
+    <joint name="world-to-base" type="fixed">
         <!-- The base of the arm is at 0,0,0 -->
         <origin xyz="0.5 0.5 0" rpy="0 0 0"/>
@@ -20,7 +26,7 @@
         <visual>
             <!-- start slightly offset, so link is at base of cylinder -->
-            <origin xyz="0 0 0.05" rpy="0 0 0"/>
+            <origin xyz="0 0 0.75" rpy="0 0 0"/>
             <geometry>
-                <cylinder length="0.1" radius="0.5"/>
+                <box size="2 2 1.5"/>
             </geometry>
             <material name="white"/>
@@ -28,8 +34,8 @@
     </link>
     <!-- http://wiki.ros.org/urdf/XML/joint -->
-    <joint name="base-to-section1" type="revolute">
-        <origin xyz="0 0 0.1"/>
+    <joint name="base-to-circle" type="revolute">
+        <origin xyz="0 0 1.5"/>
         <parent link="base"/>
-        <child link="section1"/>
+        <child link="circle"/>
         <!-- axis of rotation, normalized -->
         <axis xyz="0 0 1"/>
@@ -40,10 +46,43 @@
         <limit lower="0" upper="3.14159" effort="100" velocity="100"/>
     </joint>
-    <link name="section1">
+    <!-- TODO Should really come up with a better name for this part... -->
+    <!-- Represents the 'circle' piece that sits above the base of the robot arm -->
+    <link name="circle">
         <visual>
             <!-- start slightly offset, so link is at base of cylinder -->
-            <origin xyz="0 0 0.5" rpy="0 0 0"/>
+            <origin xyz="0 0 0.0625" rpy="0 0 0"/>
             <geometry>
-                <box size="0.5 0.25 1"/>
+                <cylinder radius="0.75" length="0.125"/>
+            </geometry>
+            <material name="blue"/>
+        </visual>
+    </link>
+    <joint name="circle-to-s0" type="fixed">
+        <parent link="circle"/>
+        <child link="s0"/>
+        <origin xyz="0 0 0.0625"/>
+    </joint>
+    <link name="s0">
+        <visual>
+            <origin xyz="0 0 0.25"/>
+            <geometry>
+                <box size="0.5 1.25 0.5"/>
+            </geometry>
+            <material name="red"/>
+        </visual>
+    </link>
+    <!-- The first real "arm" servo -->
+    <joint name="s0-to-s1" type="revolute">
+        <parent link="s0"/>
+        <child link="s1"/>
+        <origin xyz="0 0 0.25"/>
+        <axis xyz="0 -1 0"/>
+        <limit lower="0" upper="3.14159" effort="100" velocity="100"/>
+    </joint>
+    <link name="s1">
+        <visual>
+            <origin xyz="1.5 0 0"/>
+            <geometry>
+                <box size="3 1.25 0.5"/>
             </geometry>
             <material name="white"/>

Commit message: Added second linkage to arm, and modified arm so that center (all joints 0deg) is straight up, and each goes from -pi/2 to pi/2

File: description/arm.urdf.xacro (robot description, xacro)
@@ -44,5 +44,5 @@
         something like "${pi}" is possible but this is just a
         simple test for now... -->
-        <limit lower="0" upper="3.14159" effort="100" velocity="100"/>
+        <limit lower="-1.570796" upper="1.570796" effort="100" velocity="100"/>
     </joint>
     <!-- TODO Should really come up with a better name for this part... -->
@@ -78,14 +78,30 @@
         <origin xyz="0 0 0.25"/>
         <axis xyz="0 -1 0"/>
-        <limit lower="0" upper="3.14159" effort="100" velocity="100"/>
+        <limit lower="-1.570796" upper="1.570796" effort="100" velocity="100"/>
     </joint>
     <link name="s1">
         <visual>
-            <origin xyz="1.5 0 0"/>
+            <origin xyz="0 0 1.5"/>
             <geometry>
-                <box size="3 1.25 0.5"/>
+                <box size="0.5 1.25 3"/>
             </geometry>
             <material name="white"/>
         </visual>
     </link>
+    <joint name="s1-to-s2" type="revolute">
+        <parent link="s1"/>
+        <child link="s2"/>
+        <origin xyz="0 0 3"/>
+        <axis xyz="0 -1 0"/>
+        <limit lower="-1.570796" upper="1.570796" effort="100" velocity="100"/>
+    </joint>
+    <link name="s2">
+        <visual>
+            <origin xyz="0 0 1.5"/>
+            <geometry>
+                <box size="0.5 1.25 3"/>
+            </geometry>
+            <material name="blue"/>
+        </visual>
+    </link>
 </robot>

Commit message: Lazily added third arm section with copy paste of previous

File: description/arm.urdf.xacro (robot description, xacro)
@@ -105,3 +105,19 @@
         </visual>
     </link>
+    <joint name="s2-to-s3" type="revolute">
+        <parent link="s2"/>
+        <child link="s3"/>
+        <origin xyz="0 0 3"/>
+        <axis xyz="0 -1 0"/>
+        <limit lower="-1.570796" upper="1.570796" effort="100" velocity="100"/>
+    </joint>
+    <link name="s3">
+        <visual>
+            <origin xyz="0 0 1.5"/>
+            <geometry>
+                <box size="0.5 1.25 3"/>
+            </geometry>
+            <material name="red"/>
+        </visual>
+    </link>
 </robot>

Commit message: Arm completed in a 'bare bones' sense, still needs gazebo integration, and mass estimations

File: description/arm.urdf.xacro (robot description, xacro)
@@ -86,6 +86,5 @@
                 <box size="0.5 1.25 3"/>
             </geometry>
-            <material name="white"/>
-        </visual>
+            <material name="white"/> </visual>
     </link>
     <joint name="s1-to-s2" type="revolute">
@@ -121,3 +120,19 @@
         </visual>
     </link>
+    <joint name="gripper" type="revolute">
+        <parent link="s3"/>
+        <child link="grip-stick"/>
+        <origin xyz="0 0 3"/>
+        <axis xyz="0 0 1"/>
+        <limit lower="-1.570796" upper="1.570796" effort="100" velocity="100"/>
+    </joint>
+    <link name="grip-stick">
+        <visual>
+            <origin xyz="0 0.5 0.125" rpy="1.570796 0 0"/>  <!-- 'grip sticks' radius is offset -->
+            <geometry>
+                <cylinder length="1" radius="0.125"/>
+            </geometry>
+            <material name="white"/>
+        </visual>
+    </link>
 </robot>

Commit message: Using macro for servos, since they are pretty much 'all the same'

File: description/arm.urdf.xacro (robot description, xacro)
@@ -1,4 +1,18 @@
 <?xml version="1.0"?>
 <robot xmlns:xacro="http://www.ros.org/wiki/xacro" name="robot">
+<xacro:macro name="microServo" params="parent child origin axis">
+    <joint name="${parent}-to-${child}-servo" type="revolute">
+        <origin xyz="${origin}"/>
+        <parent link="${parent}"/>
+        <child link="${child}"/>
+        <!-- axis of rotation, normalized -->
+        <axis xyz="${axis}"/>
+        <!-- limits of rotation (in radians) and movement -->
+        <!-- TODO it might be nice to figure out how to 'macro' pi
+        something like "${pi}" is possible but this is just a
+        simple test for now... -->
+        <limit lower="-1.570796" upper="1.570796" effort="100" velocity="100"/>
+    </joint>
+</xacro:macro>
     <material name="white">
         <color rgba="1 1 1 1"/>
@@ -12,5 +26,4 @@
     <!-- Base link, true, non-relative 0,0,0 of world -->
     <link name="world"></link>
-    <!-- connection from the world, to the base of the arm-->
     <joint name="world-to-base" type="fixed">
         <!-- The base of the arm is at 0,0,0 -->
@@ -20,7 +33,7 @@
         <!-- the 'child' link, or next in heirarchy -->
         <child link="base"/>
-        <!-- <limit /> -->
     </joint>
     <!-- the "Base" of the robotic arm -->
+    <xacro:property name="base_dimensions" value="2 2 1.5"/>
     <link name="base">
         <visual>
@@ -28,22 +41,10 @@
             <origin xyz="0 0 0.75" rpy="0 0 0"/>
             <geometry>
-                <box size="2 2 1.5"/>
+                <box size="${base_dimensions}"/>
             </geometry>
-            <material name="white"/>
+            <material name="red"/>
         </visual>
     </link>
-    <!-- http://wiki.ros.org/urdf/XML/joint -->
-    <joint name="base-to-circle" type="revolute">
-        <origin xyz="0 0 1.5"/>
-        <parent link="base"/>
-        <child link="circle"/>
-        <!-- axis of rotation, normalized -->
-        <axis xyz="0 0 1"/>
-        <!-- limits of rotation (in radians) and movement -->
-        <!-- TODO it might be nice to figure out how to 'macro' pi
-        something like "${pi}" is possible but this is just a
-        simple test for now... -->
-        <limit lower="-1.570796" upper="1.570796" effort="100" velocity="100"/>
-    </joint>
+    <xacro:microServo parent="base" child="circle" origin="0 0 1.5" axis="0 0 1"/>
     <!-- TODO Should really come up with a better name for this part... -->
     <!-- Represents the 'circle' piece that sits above the base of the robot arm -->
@@ -63,4 +64,6 @@
         <origin xyz="0 0 0.0625"/>
     </joint>
+    <!-- representation of base of the arm -->
+    <!-- between the circle and first real arm segment s1 -->
     <link name="s0">
         <visual>
@@ -72,12 +75,6 @@
         </visual>
     </link>
-    <!-- The first real "arm" servo -->
-    <joint name="s0-to-s1" type="revolute">
-        <parent link="s0"/>
-        <child link="s1"/>
-        <origin xyz="0 0 0.25"/>
-        <axis xyz="0 -1 0"/>
-        <limit lower="-1.570796" upper="1.570796" effort="100" velocity="100"/>
-    </joint>
+    <!-- The first real "arm" servo, may want to be +1 instead but will have to update servo code?-->
+    <xacro:microServo parent="s0" child="s1" origin="0 0 0.25" axis="0 -1 0"/>
     <link name="s1">
         <visual>
@@ -86,13 +83,8 @@
                 <box size="0.5 1.25 3"/>
             </geometry>
-            <material name="white"/> </visual>
+            <material name="white"/>
+        </visual>
     </link>
-    <joint name="s1-to-s2" type="revolute">
-        <parent link="s1"/>
-        <child link="s2"/>
-        <origin xyz="0 0 3"/>
-        <axis xyz="0 -1 0"/>
-        <limit lower="-1.570796" upper="1.570796" effort="100" velocity="100"/>
-    </joint>
+    <xacro:microServo parent="s1" child="s2" origin="0 0 3" axis="0 -1 0"/>
     <link name="s2">
         <visual>
@@ -104,11 +96,5 @@
         </visual>
     </link>
-    <joint name="s2-to-s3" type="revolute">
-        <parent link="s2"/>
-        <child link="s3"/>
-        <origin xyz="0 0 3"/>
-        <axis xyz="0 -1 0"/>
-        <limit lower="-1.570796" upper="1.570796" effort="100" velocity="100"/>
-    </joint>
+    <xacro:microServo parent="s2" child="s3" origin="0 0 3" axis="0 -1 0"/>
     <link name="s3">
         <visual>
@@ -120,11 +106,5 @@
         </visual>
     </link>
-    <joint name="gripper" type="revolute">
-        <parent link="s3"/>
-        <child link="grip-stick"/>
-        <origin xyz="0 0 3"/>
-        <axis xyz="0 0 1"/>
-        <limit lower="-1.570796" upper="1.570796" effort="100" velocity="100"/>
-    </joint>
+    <xacro:microServo parent="s3" child="grip-stick" origin="0 0 3" axis="0 0 1"/>
     <link name="grip-stick">
         <visual>

Commit message: links for main arm macro'd

File: description/arm.urdf.xacro (robot description, xacro)
@@ -14,4 +14,15 @@
         <limit lower="-1.570796" upper="1.570796" effort="100" velocity="100"/>
     </joint>
+</xacro:macro>
+<xacro:macro name="arm-segment" params="number origin size material">
+    <link name="s${number}">
+        <visual>
+            <origin xyz="${origin}"/>
+            <geometry>
+                <box size="${size}"/>
+            </geometry>
+            <material name="${material}"/>
+        </visual>
+    </link>
 </xacro:macro>
     <material name="white">
@@ -77,33 +88,9 @@
     <!-- The first real "arm" servo, may want to be +1 instead but will have to update servo code?-->
     <xacro:microServo parent="s0" child="s1" origin="0 0 0.25" axis="0 -1 0"/>
-    <link name="s1">
-        <visual>
-            <origin xyz="0 0 1.5"/>
-            <geometry>
-                <box size="0.5 1.25 3"/>
-            </geometry>
-            <material name="white"/>
-        </visual>
-    </link>
+    <xacro:arm-segment number="1" origin="0 0 1.5" size="0.5 1.25 3" material="white"/>
     <xacro:microServo parent="s1" child="s2" origin="0 0 3" axis="0 -1 0"/>
-    <link name="s2">
-        <visual>
-            <origin xyz="0 0 1.5"/>
-            <geometry>
-                <box size="0.5 1.25 3"/>
-            </geometry>
-            <material name="blue"/>
-        </visual>
-    </link>
+    <xacro:arm-segment number="2" origin="0 0 1.5" size="0.5 1.25 3" material="blue"/>
     <xacro:microServo parent="s2" child="s3" origin="0 0 3" axis="0 -1 0"/>
-    <link name="s3">
-        <visual>
-            <origin xyz="0 0 1.5"/>
-            <geometry>
-                <box size="0.5 1.25 3"/>
-            </geometry>
-            <material name="red"/>
-        </visual>
-    </link>
+    <xacro:arm-segment number="3" origin="0 0 1.5" size="0.5 1.25 3" material="red"/>
     <xacro:microServo parent="s3" child="grip-stick" origin="0 0 3" axis="0 0 1"/>
     <link name="grip-stick">

Commit message: Updated to use a seprate macro file

File: description/arm.urdf.xacro (robot description, xacro)
@@ -1,38 +1,5 @@
 <?xml version="1.0"?>
 <robot xmlns:xacro="http://www.ros.org/wiki/xacro" name="robot">
-<xacro:macro name="microServo" params="parent child origin axis">
-    <joint name="${parent}-to-${child}-servo" type="revolute">
-        <origin xyz="${origin}"/>
-        <parent link="${parent}"/>
-        <child link="${child}"/>
-        <!-- axis of rotation, normalized -->
-        <axis xyz="${axis}"/>
-        <!-- limits of rotation (in radians) and movement -->
-        <!-- TODO it might be nice to figure out how to 'macro' pi
-        something like "${pi}" is possible but this is just a
-        simple test for now... -->
-        <limit lower="-1.570796" upper="1.570796" effort="100" velocity="100"/>
-    </joint>
-</xacro:macro>
-<xacro:macro name="arm-segment" params="number origin size material">
-    <link name="s${number}">
-        <visual>
-            <origin xyz="${origin}"/>
-            <geometry>
-                <box size="${size}"/>
-            </geometry>
-            <material name="${material}"/>
-        </visual>
-    </link>
-</xacro:macro>
-    <material name="white">
-        <color rgba="1 1 1 1"/>
-    </material>
-    <material name="blue">
-        <color rgba="0 0 1 1"/>
-    </material>
-    <material name="red">
-        <color rgba="1 0 0 1"/>
-    </material>
+    <xacro:include filename="macros.urdf.xacro"/>
     <!-- Base link, true, non-relative 0,0,0 of world -->
     <link name="world"></link>
@@ -54,8 +21,7 @@
                 <box size="${base_dimensions}"/>
             </geometry>
-            <material name="red"/>
+            <material name="cyan"/>
         </visual>
     </link>
-    <xacro:microServo parent="base" child="circle" origin="0 0 1.5" axis="0 0 1"/>
     <!-- TODO Should really come up with a better name for this part... -->
     <!-- Represents the 'circle' piece that sits above the base of the robot arm -->
@@ -75,4 +41,10 @@
         <origin xyz="0 0 0.0625"/>
     </joint>
+    <!-- The first real "arm" servo, may want to be +1 instead but will have to update servo code?-->
+    <xacro:microServo parent="base" child="circle" origin="0 0 1.5" axis="0 0 1"/>
+    <xacro:microServo parent="s0" child="s1" origin="0 0 0.25" axis="0 -1 0"/>
+    <xacro:microServo parent="s2" child="s3" origin="0 0 3" axis="0 -1 0"/>
+    <xacro:microServo parent="s3" child="grip-stick" origin="0 0 3" axis="0 0 1"/>
+    <xacro:microServo parent="s1" child="s2" origin="0 0 3" axis="0 -1 0"/>
     <!-- representation of base of the arm -->
     <!-- between the circle and first real arm segment s1 -->
@@ -86,12 +58,7 @@
         </visual>
     </link>
-    <!-- The first real "arm" servo, may want to be +1 instead but will have to update servo code?-->
-    <xacro:microServo parent="s0" child="s1" origin="0 0 0.25" axis="0 -1 0"/>
     <xacro:arm-segment number="1" origin="0 0 1.5" size="0.5 1.25 3" material="white"/>
-    <xacro:microServo parent="s1" child="s2" origin="0 0 3" axis="0 -1 0"/>
     <xacro:arm-segment number="2" origin="0 0 1.5" size="0.5 1.25 3" material="blue"/>
-    <xacro:microServo parent="s2" child="s3" origin="0 0 3" axis="0 -1 0"/>
     <xacro:arm-segment number="3" origin="0 0 1.5" size="0.5 1.25 3" material="red"/>
-    <xacro:microServo parent="s3" child="grip-stick" origin="0 0 3" axis="0 0 1"/>
     <link name="grip-stick">
         <visual>
@@ -103,3 +70,9 @@
         </visual>
     </link>
+    <!-- Link in gazebo -->
+    <gazebo>
+        <plugin name="gazebo_ros_control" filename="libgazebo_ros_control.so">
+            <robotNamespace>/</robotNamespace>
+        </plugin>
+    </gazebo>
 </robot>

Commit message: added collision tags matching all the box tags

File: description/arm.urdf.xacro (robot description, xacro)
@@ -1,5 +1,5 @@
 <?xml version="1.0"?>
 <robot xmlns:xacro="http://www.ros.org/wiki/xacro" name="robot">
-    <xacro:include filename="macros.urdf.xacro"/>
+    <xacro:include filename="macros.xacro"/>
     <!-- Base link, true, non-relative 0,0,0 of world -->
     <link name="world"></link>
@@ -35,4 +35,11 @@
             <material name="blue"/>
         </visual>
+        <collision>
+            <!-- start slightly offset, so link is at base of cylinder -->
+            <origin xyz="0 0 0.0625" rpy="0 0 0"/>
+            <geometry>
+                <cylinder radius="0.75" length="0.125"/>
+            </geometry>
+        </collision>
     </link>
     <joint name="circle-to-s0" type="fixed">
@@ -44,7 +51,7 @@
     <xacro:microServo parent="base" child="circle" origin="0 0 1.5" axis="0 0 1"/>
     <xacro:microServo parent="s0" child="s1" origin="0 0 0.25" axis="0 -1 0"/>
+    <xacro:microServo parent="s1" child="s2" origin="0 0 3" axis="0 -1 0"/>
     <xacro:microServo parent="s2" child="s3" origin="0 0 3" axis="0 -1 0"/>
     <xacro:microServo parent="s3" child="grip-stick" origin="0 0 3" axis="0 0 1"/>
-    <xacro:microServo parent="s1" child="s2" origin="0 0 3" axis="0 -1 0"/>
     <!-- representation of base of the arm -->
     <!-- between the circle and first real arm segment s1 -->
@@ -52,9 +59,11 @@
         <visual>
             <origin xyz="0 0 0.25"/>
-            <geometry>
-                <box size="0.5 1.25 0.5"/>
-            </geometry>
+            <geometry> <box size="0.5 1.25 0.5"/> </geometry>
             <material name="red"/>
         </visual>
+        <collision>
+            <origin xyz="0 0 0.25"/>
+            <geometry> <box size="0.5 1.25 0.5"/> </geometry>
+        </collision>
     </link>
     <xacro:arm-segment number="1" origin="0 0 1.5" size="0.5 1.25 3" material="white"/>
@@ -64,11 +73,15 @@
         <visual>
             <origin xyz="0 0.5 0.125" rpy="1.570796 0 0"/>  <!-- 'grip sticks' radius is offset -->
-            <geometry>
-                <cylinder length="1" radius="0.125"/>
-            </geometry>
+            <geometry> <cylinder length="1" radius="0.125"/> </geometry>
             <material name="white"/>
         </visual>
+        <collision>
+            <origin xyz="0 0.5 0.125" rpy="1.570796 0 0"/>  <!-- 'grip sticks' radius is offset -->
+            <geometry> <cylinder length="1" radius="0.125"/> </geometry>
+        </collision>
     </link>
     <!-- Link in gazebo -->
+    <xacro:include filename="gazebo.xacro"/>
+    <!--
     <gazebo>
         <plugin name="gazebo_ros_control" filename="libgazebo_ros_control.so">
@@ -76,3 +89,4 @@
         </plugin>
     </gazebo>
+    -->
 </robot>
