Commit message: Robot arm appears in gazebo! just not well or right

File: description/arm.urdf.xacro (robot description, xacro)
@@ -13,9 +13,12 @@
     </joint>
     <!-- the "Base" of the robotic arm -->
-    <xacro:property name="base_dimensions" value="2 2 1.5"/>
+    <xacro:property name="base_x" value="2"/>
+    <xacro:property name="base_y" value="2"/>
+    <xacro:property name="base_z" value="1.5"/>
+    <xacro:property name="base_dimensions" value="${base_x} ${base_y} ${base_z}"/>
+    <xacro:property name="base_origin" value="0 0 0.75"/>
     <link name="base">
         <visual>
-            <!-- start slightly offset, so link is at base of cylinder -->
-            <origin xyz="0 0 0.75" rpy="0 0 0"/>
+            <origin xyz="${base_origin}"/>
             <geometry>
                 <box size="${base_dimensions}"/>
@@ -23,13 +26,26 @@
             <material name="cyan"/>
         </visual>
+        <collision>
+            <origin xyz="${base_origin}"/>
+            <geometry>
+                <box size="${base_dimensions}"/>
+            </geometry>
+        </collision>
+        <xacro:inertial_box mass="2" x="${base_x}" y="${base_y}"  z="${base_z}">
+            <origin xyz="${base_origin}"/>
+        </xacro:inertial_box>
     </link>
     <!-- TODO Should really come up with a better name for this part... -->
     <!-- Represents the 'circle' piece that sits above the base of the robot arm -->
+    <xacro:property name="circle_height" value="0.125"/>
+    <xacro:property name="circle_radius" value="0.75"/>
+    <!-- TODO this should probably be different? not the cleanest way to do it -->
+    <xacro:property name="circle_origin" value="0 0 0.0625"/>
     <link name="circle">
         <visual>
             <!-- start slightly offset, so link is at base of cylinder -->
-            <origin xyz="0 0 0.0625" rpy="0 0 0"/>
+            <origin xyz="${circle_origin}" rpy="0 0 0"/>
             <geometry>
-                <cylinder radius="0.75" length="0.125"/>
+                <cylinder radius="${circle_radius}" length="${circle_height}"/>
             </geometry>
             <material name="blue"/>
@@ -37,9 +53,12 @@
         <collision>
             <!-- start slightly offset, so link is at base of cylinder -->
-            <origin xyz="0 0 0.0625" rpy="0 0 0"/>
+            <origin xyz="${circle_origin}" rpy="0 0 0"/>
             <geometry>
-                <cylinder radius="0.75" length="0.125"/>
+                <cylinder radius="${circle_radius}" length="${circle_height}"/>
             </geometry>
         </collision>
+        <xacro:inertial_cylinder mass="0.1" length="${circle_height}" radius="${circle_radius}">
+            <origin xyz="${circle_origin}"/>
+        </xacro:inertial_cylinder>
     </link>
     <joint name="circle-to-s0" type="fixed">
@@ -53,40 +72,51 @@
     <xacro:microServo parent="s1" child="s2" origin="0 0 3" axis="0 -1 0"/>
     <xacro:microServo parent="s2" child="s3" origin="0 0 3" axis="0 -1 0"/>
-    <xacro:microServo parent="s3" child="grip-stick" origin="0 0 3" axis="0 0 1"/>
+    <xacro:microServo parent="s3" child="grip_stick" origin="0 0 3" axis="0 0 1"/>
     <!-- representation of base of the arm -->
     <!-- between the circle and first real arm segment s1 -->
+    <xacro:property name="s0_origin" value="0 0 0.25"/>
+    <xacro:property name="s0xLen" value="0.5"/>
+    <xacro:property name="s0yLen" value="1.25"/>
+    <xacro:property name="s0zLen" value="0.5"/>
     <link name="s0">
         <visual>
-            <origin xyz="0 0 0.25"/>
-            <geometry> <box size="0.5 1.25 0.5"/> </geometry>
+            <origin xyz="${s0_origin}"/>
+            <geometry> <box size="${s0xLen} ${s0yLen} ${s0zLen}"/> </geometry>
             <material name="red"/>
         </visual>
         <collision>
-            <origin xyz="0 0 0.25"/>
-            <geometry> <box size="0.5 1.25 0.5"/> </geometry>
+            <origin xyz="${s0_origin}"/>
+            <geometry> <box size="${s0xLen} ${s0yLen} ${s0zLen}"/> </geometry>
         </collision>
+        <xacro:inertial_box mass="0.1" x="${s0xLen}" y="${s0yLen}" z="${s0zLen}">
+            <origin xyz="${s0_origin}"/>
+        </xacro:inertial_box>
     </link>
-    <xacro:arm-segment number="1" origin="0 0 1.5" size="0.5 1.25 3" material="white"/>
-    <xacro:arm-segment number="2" origin="0 0 1.5" size="0.5 1.25 3" material="blue"/>
-    <xacro:arm-segment number="3" origin="0 0 1.5" size="0.5 1.25 3" material="red"/>
-    <link name="grip-stick">
+    <xacro:arm-segment number="1" origin="0 0 1.5" x="0.5" y="1.25" z="3" material="white"/>
+    <xacro:arm-segment number="2" origin="0 0 1.5" x="0.5" y="1.25" z="3" material="red"/>
+    <xacro:arm-segment number="3" origin="0 0 1.5" x="0.5" y="1.25" z="3" material="blue"/>
+    <xacro:property name="grip_stick_height" value="1"/>
+    <xacro:property name="grip_stick_radius" value="0.75"/>
+    <xacro:property name="grip_stick_origin" value="0 0.5 0.125"/>
+    <xacro:property name="grip_stick_rpy" value="1.572 0 0"/>
+    <link name="grip_stick">
         <visual>
-            <origin xyz="0 0.5 0.125" rpy="1.570796 0 0"/>  <!-- 'grip sticks' radius is offset -->
-            <geometry> <cylinder length="1" radius="0.125"/> </geometry>
+            <origin xyz="${grip_stick_origin}" rpy="${grip_stick_rpy}"/>  <!-- 'grip sticks' radius is offset -->
+            <geometry>
+                <cylinder length="${grip_stick_height}" radius="${grip_stick_radius}"/>
+            </geometry>
             <material name="white"/>
         </visual>
         <collision>
-            <origin xyz="0 0.5 0.125" rpy="1.570796 0 0"/>  <!-- 'grip sticks' radius is offset -->
-            <geometry> <cylinder length="1" radius="0.125"/> </geometry>
+            <origin xyz="${grip_stick_origin}" rpy="${grip_stick_rpy}"/>  <!-- 'grip sticks' radius is offset -->
+            <geometry>
+                <cylinder length="${grip_stick_height}" radius="${grip_stick_radius}"/>
+            </geometry>
         </collision>
+        <xacro:inertial_cylinder mass="0.25" length="${grip_stick_height}" radius="${grip_stick_radius}">
+            <origin xyz="${grip_stick_origin}" rpy="${grip_stick_rpy}"/>  <!-- 'grip sticks' radius is offset -->
+        </xacro:inertial_cylinder>
     </link>
-    <!-- Link in gazebo -->
+    <!-- Link in gazebo file, which contains all of hte gazebo related things -->
     <xacro:include filename="gazebo.xacro"/>
-    <!--
-    <gazebo>
-        <plugin name="gazebo_ros_control" filename="libgazebo_ros_control.so">
-            <robotNamespace>/</robotNamespace>
-        </plugin>
-    </gazebo>
-    -->
 </robot>

File: description/macros.xacro (robot description, xacro)
@@ -37,16 +37,37 @@
         </transmission> -->
     </xacro:macro>
-    <xacro:macro name="arm-segment" params="number origin size material">
+    <xacro:macro name="arm-segment" params="number origin x y z material">
         <link name="s${number}">
             <visual>
                 <origin xyz="${origin}"/>
-                <geometry> <box size="${size}"/> </geometry>
+                <geometry> <box size="${x} ${y} ${z}"/> </geometry>
                 <material name="${material}"/>
             </visual>
             <collision>
                 <origin xyz="${origin}"/>
-                <geometry> <box size="${size}"/> </geometry>
+                <geometry> <box size="${x} ${y} ${z}"/> </geometry>
             </collision>
+            <xacro:inertial_box mass="1" x="${x}" y="${y}" z="${z}">
+                <origin xyz="${origin}"/>
+            </xacro:inertial_box>
         </link>
     </xacro:macro>
+    <xacro:macro name="inertial_box" params="mass x y z *origin">
+        <inertial>
+            <xacro:insert_block name="origin"/>
+            <mass value="${mass}" />
+            <inertia ixx="${(1/12) * mass * (y*y+z*z)}" ixy="0.0" ixz="0.0"
+                    iyy="${(1/12) * mass * (x*x+z*z)}" iyz="0.0"
+                    izz="${(1/12) * mass * (x*x+y*y)}" />
+        </inertial>
+    </xacro:macro>
+    <xacro:macro name="inertial_cylinder" params="mass length radius *origin">
+        <inertial>
+            <xacro:insert_block name="origin"/>
+            <mass value="${mass}" />
+            <inertia ixx="${(1/12) * mass * (3*radius*radius + length*length)}" ixy="0.0" ixz="0.0"
+                    iyy="${(1/12) * mass * (3*radius*radius + length*length)}" iyz="0.0"
+                    izz="${(1/2) * mass * (radius*radius)}" />
+        </inertial>
+    </xacro:macro>
 </robot>

Commit message: Gave arm colors and cleaned up

File: description/arm.urdf.xacro (robot description, xacro)
@@ -97,5 +97,5 @@
     <xacro:arm-segment number="3" origin="0 0 1.5" x="0.5" y="1.25" z="3" material="blue"/>
     <xacro:property name="grip_stick_height" value="1"/>
-    <xacro:property name="grip_stick_radius" value="0.75"/>
+    <xacro:property name="grip_stick_radius" value="0.075"/>
     <xacro:property name="grip_stick_origin" value="0 0.5 0.125"/>
     <xacro:property name="grip_stick_rpy" value="1.572 0 0"/>

File: description/gazebo.xacro (robot description, xacro)
@@ -1,11 +1,25 @@
 <?xml version="1.0"?>
 <robot xmlns:xacro="http://www.ros.org/wiki/xacro">
-    <!-- All gazebo stuff will go here -->
-    <!--  May need this?
-    <gazebo>
-        <plugin name="gazebo_ros_control" filename="libgazebo_ros_control.so">
-            <robotNamespace>/</robotNamespace>
-        </plugin>
+    <!-- Give it color in gazebo -->
+    <gazebo reference='base'>
+        <material>Gazebo/Red</material>
     </gazebo>
-    -->
+    <gazebo reference='circle'>
+        <material>Gazebo/White</material>
+    </gazebo>
+    <gazebo reference='s0'>
+        <material>Gazebo/Blue</material>
+    </gazebo>
+    <gazebo reference='s1'>
+        <material>Gazebo/Red</material>
+    </gazebo>
+    <gazebo reference='s2'>
+        <material>Gazebo/White</material>
+    </gazebo>
+    <gazebo reference='s3'>
+        <material>Gazebo/Blue</material>
+    </gazebo>
+    <gazebo reference='grip_stick'>
+        <material>Gazebo/Red</material>
+    </gazebo>
 </robot>

File: description/macros.xacro (robot description, xacro)
@@ -14,5 +14,5 @@
     </material>
     <xacro:macro name="microServo" params="parent child origin axis">
-        <joint name="${parent}-to-${child}-servo" type="revolute">
+        <joint name="${parent}_${child}_servo" type="revolute">
             <origin xyz="${origin}"/>
             <parent link="${parent}"/>

Commit message: Whatever I had at the end of last semester, INCOMPLETE, PROBABLY BROKEN

File: description/arm.urdf.xacro (robot description, xacro)
@@ -2,4 +2,6 @@
 <robot xmlns:xacro="http://www.ros.org/wiki/xacro" name="robot">
     <xacro:include filename="macros.xacro"/>
+    <!-- Link in gazebo file, which contains all of hte gazebo related things -->
+    <xacro:include filename="gazebo.xacro"/>
     <!-- Base link, true, non-relative 0,0,0 of world -->
     <link name="world"></link>
@@ -36,9 +38,7 @@
         </xacro:inertial_box>
     </link>
-    <!-- TODO Should really come up with a better name for this part... -->
     <!-- Represents the 'circle' piece that sits above the base of the robot arm -->
     <xacro:property name="circle_height" value="0.125"/>
     <xacro:property name="circle_radius" value="0.75"/>
-    <!-- TODO this should probably be different? not the cleanest way to do it -->
     <xacro:property name="circle_origin" value="0 0 0.0625"/>
     <link name="circle">
@@ -118,5 +118,3 @@
         </xacro:inertial_cylinder>
     </link>
-    <!-- Link in gazebo file, which contains all of hte gazebo related things -->
-    <xacro:include filename="gazebo.xacro"/>
 </robot>

File: description/gazebo.xacro (robot description, xacro)
@@ -1,5 +1,4 @@
 <?xml version="1.0"?>
 <robot xmlns:xacro="http://www.ros.org/wiki/xacro">
-    <!-- Give it color in gazebo -->
     <gazebo reference='base'>
         <material>Gazebo/Red</material>

File: description/macros.xacro (robot description, xacro)
@@ -26,14 +26,4 @@
             <limit lower="-1.570796" upper="1.570796" effort="100" velocity="100"/>
         </joint>
-        <!--
-        <transmission name="${parent}-${child}-servo-trans">
-            <type>transmission_interface/SimpleTransmission</type>
-            <actuator name="${parent}-to-${child}">
-              <mechanicalReduction>1</mechanicalReduction>
-            </actuator>
-            <joint name="${parent}-to-${child}-servo">
-              <hardwareInterface>hardware_interface/PositionJointInterface</hardwareInterface>
-            </joint>
-        </transmission> -->
     </xacro:macro>
     <xacro:macro name="arm-segment" params="number origin x y z material">
